File: Hackpad PCB/Hackpad.kicad_sch (KiCad schematic)
At the start: 37 parts, among them SW1 SW_Push, SW10 RotaryEncoder_Switch, SW2 SW_Push, SW3 SW_Push, SW4 SW_Push, SW5 SW_Push, SW6 SW_Push, SW7 SW_Push, SW8 SW_Push, SW9 SW_Push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

Commit message: Add BOM
Parts:
- renumbered SW10 to SW13
Changed lines of the file:
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@@
 		(dnp no)
 		(fields_autoplaced yes)
-		(property "Reference" "SW10"
+		(property "Reference" "SW13"
 			(at 107.95 139.7 0)
 			(effects
@@
 			(project ""
 				(path "/003a1ca2-44ae-475f-9cc4-8f1a70aac36d"
-					(reference "SW10")
+					(reference "SW13")
 					(unit 1)
 				)
